File: board/hugo_board/hugo_board.kicad_sch (KiCad schematic)
At the start: 22 parts, among them J1 Screw_Terminal_01x02, J10 Screw_Terminal_01x02, J2 Screw_Terminal_01x02, J3 Screw_Terminal_01x02, J4 Screw_Terminal_01x02, J5 Screw_Terminal_01x02, J6 Screw_Terminal_01x02, J7 Screw_Terminal_01x02, J8 Screw_Terminal_01x02, J9 Screw_Terminal_01x02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

Commit message: version 2
Parts:
- removed J1, J10, J2, J3, J4, J5, J6, J8, J9: Screw_Terminal_01x02, TerminalBlock_4Ucon:TerminalBlock_4Ucon_1x02_P3.50mm_Vertical, symbol Connector:Screw_Terminal_01x02
- added BLUE1, BLUE2, BLUE3, GREEN1, GREEN2, GREEN3, RED1, RED2, RED3: LED, LED_THT:LED_D10.0mm, symbol Device:LED
- SW1, SW2, SW3: footprint TerminalBlock_4Ucon:TerminalBlock_4Ucon_1x02_P3.50mm_Vertical -> TerminalBlock_4Ucon:TerminalBlock_4Ucon_1x02_P3.50mm_Horizontal
- renumbered J7 to J1
Connections:
- net +BATT: now also BLUE1.1 (K), BLUE2.1 (K), BLUE3.1 (K), GREEN1.1 (K), GREEN2.1 (K), GREEN3.1 (K), RED1.1 (K), RED2.1 (K), RED3.1 (K)
- net at R7.1: now also GREEN1.2 (A)
- net at R9.1: now also GREEN3.2 (A)
- net at R4.1: now also RED1.2 (A)
- net at R5.1: now also RED2.2 (A)
- net at R6.1: now also RED3.2 (A)
- net at R8.1: now also GREEN2.2 (A)
- net at R2.1: now also BLUE2.2 (A)
- net at R1.1: now also BLUE1.2 (A)
- net at R3.1: now also BLUE3.2 (A)
